Commit message: Repair urdf parts for irb1400

File: urdf_models/urdf/base.urdf (robot description, URDF)
Before this commit: robot base, 1 links, 0 joints
Links:
- removed link base_with_coordinate_system
- added link base, mass 25.417; collision mesh filename=package://urdf_models/meshes/base.STL; visual mesh filename=package://urdf_models/meshes/base.STL

File: urdf_models/urdf/link1.urdf (robot description, URDF)
Before this commit: robot link1, 1 links, 0 joints
Links:
- removed link link1_fixed_coordinate
- added link link1, mass 32.007; collision mesh filename=package://urdf_models/meshes/link1.STL; visual mesh filename=package://urdf_models/meshes/link1.STL

File: urdf_models/urdf/link2.urdf (robot description, URDF)
Before this commit: robot link2, 1 links, 0 joints
Links:
- removed link link2_fixed_coordinate
- added link link2, mass 7.6192; collision mesh filename=package://urdf_models/meshes/link2.STL; visual mesh filename=package://urdf_models/meshes/link2.STL

File: urdf_models/urdf/link3.urdf (robot description, URDF)
Before this commit: robot link3, 1 links, 0 joints
Links:
- removed link link3_fixed_coordinate
- added link link3, mass 7.4487; collision mesh filename=package://urdf_models/meshes/link3.STL; visual mesh filename=package://urdf_models/meshes/link3.STL

File: urdf_models/urdf/link4.urdf (robot description, URDF)
Before this commit: robot link4, 1 links, 0 joints
Links:
- removed link link4_fixed_coordinate
- added link link4, mass 11.024; collision mesh filename=package://urdf_models/meshes/link4.STL; visual mesh filename=package://urdf_models/meshes/link4.STL

File: urdf_models/urdf/link5.urdf (robot description, URDF)
Before this commit: robot link5, 1 links, 0 joints
Links:
- removed link link5_fixed_coordinate
- added link link5, mass 0.29435; collision mesh filename=package://urdf_models/meshes/link5.STL; visual mesh filename=package://urdf_models/meshes/link5.STL

File: urdf_models/urdf/link6.urdf (robot description, URDF)
Before this commit: robot link6, 1 links, 0 joints
Links:
- removed link link6_fixed_coordinate
- added link link6, mass 0.016853; collision mesh filename=package://urdf_models/meshes/link6.STL; visual mesh filename=package://urdf_models/meshes/link6.STL

File: urdf_models/urdf/part_viewer.urdf (robot description, URDF)
Before this commit: robot irb1400, 1 links, 0 joints
Links:
- removed link link2_fixed_coordinate
- added link link4, mass 11.024; collision mesh filename=package://urdf_models/meshes/link4.STL; visual mesh filename=package://urdf_models/meshes/link4.STL
