Commit message: Debug robot_viewer

File: urdf_models/urdf/roboto.urdf (robot description, URDF)
Before this commit: robot irb1400, 2 links, 0 joints
Links:
- removed link base_with_coordinate_system
- removed link link_1
- added link base, mass 25.417; collision mesh filename=package://urdf_models/meshes/base.STL; visual mesh filename=package://urdf_models/meshes/base.STL
- added link link1, mass 32.007; collision mesh filename=package://urdf_models/meshes/link1.STL; visual mesh filename=package://urdf_models/meshes/link1.STL
- added link world
Joints:
- added joint joint1: type revolute, parent base, child link1, origin xyz=0 0 0.0925 rpy=0 0 0, axis 0 0 1, limit lower=-2.967 effort=1000.0 velocity=5
- added joint world_to_robot: type fixed, parent world, child base, origin xyz=0 0 0 rpy=0 0 0
