Commit message: Add and fixed link 1 and 4. Use link4_2nd

File: urdf_models/urdf/link1_nov9.urdf (robot description, URDF)
Before this commit: robot link4, 1 links, 0 joints
Links:
- removed link link4_2nd
- added link link1_fixed_origin_nov9, mass 32.007; collision mesh filename=package://link1_fixed_origin_nov9/meshes/link1_fixed_origin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; visual mesh filename=package://link1_fixed_origin_nov9/meshes/link1_fixed_origin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

File: urdf_models/urdf/link4_nov9.urdf (robot description, URDF)
Before this commit: robot link4, 1 links, 0 joints
Links:
- removed link link4_2nd
- added link link4_fixed_origin_nov9, mass 11.024; collision mesh filename=package://link4_fixed_origin_nov9/meshes/link4_fixed_origin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; visual mesh filename=package://link4_fixed_origin_nov9/meshes/link4_fixed_origin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
