Commit message: Modify roboto_visual.urdf for a full irb1400 robot model

File: urdf_models/urdf/roboto_visual.urdf (robot description, URDF)
Before this commit: robot roboto_visual, 3 links, 2 joints
Links:
- added link link2; visual mesh filename=package://urdf_models/meshes/link2.STL
- added link link3; visual mesh filename=package://urdf_models/meshes/link3.STL
- added link link4; visual mesh filename=package://urdf_models/meshes/link4_2nd.STL
- added link link5; visual mesh filename=package://urdf_models/meshes/link5.STL
- added link link6; visual mesh filename=package://urdf_models/meshes/link6.STL
- added link link7
Joints:
- added joint joint2: type revolute, parent link1, child link2, origin xyz=0.15 0 0.345 rpy=-1.5707 0 0, axis 0 0 1, limit lower=-2.7925 upper=0 effort=1.0 velocity=5.0
- added joint joint3: type revolute, parent link2, child link3, origin xyz=0.6 0 0 rpy=0 0 0, axis 0 0 1, limit lower=-1.5708 upper=1.5708 effort=1.0 velocity=5.0
- added joint joint4: type revolute, parent link3, child link4, origin xyz=0.12 0 0 rpy=-1.5707 0 0, axis 0 0 1, limit lower=0 upper=3.142 effort=1.0 velocity=5.0
- added joint joint5: type revolute, parent link4, child link5, origin xyz=0 0 0.72 rpy=1.5708 0 0, axis 0 0 1, limit lower=0 upper=3.142 effort=1.0 velocity=5.0
- added joint joint6: type revolute, parent link5, child link6, origin xyz=0 0 0 rpy=-1.5708 0 0, axis 0 0 1, limit lower=0 upper=3.142 effort=1.0 velocity=5.0
- added joint joint7: type fixed, parent link6, child link7, origin xyz=0 0 0.085 rpy=0 0 0
- joint joint1: limit lower=0.0 upper=1.9 effort=1.0 velocity=5.0 -> lower=-1.4835 upper=1.4835 effort=1.0 velocity=5.0; origin xyz=0 0 0.0925 rpy=0 0 0 -> xyz=0 0 0.118 rpy=0 0 0
